File: Hardware/SparkFun_Qwiic_Current_Sensor_ADE7953.kicad_pcb (KiCad board)
At the start: 2 copper layers, 25.4 x 25.4 mm, 85 parts, among them J1 Qwiic_RA, J2 Qwiic_RA, J3 Conn_01x06, J4 Conn_01x02, J5 3.5mm TRRS, J6 Conn_01x02, U1 ADE7953ACPZ, Y1 3.579MHz

Commit message: Moved R11
Parts:
- moved R11 2.56 mm to (141.0, 106.7)
Routing:
- net Net-(JP3-C): track 6.51 -> 4.74 mm
- net ~{INT}: track 12.1 -> 11.3 mm
Changed lines of the file:
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@@
 				(font
 					(size 0.001 0.001)
+					(thickness 0.15)
 				)
 			)
@@
 				(font
 					(size 0.001 0.001)
+					(thickness 0.15)
 				)
 			)
@@
 				(font
 					(size 0.001 0.001)
+					(thickness 0.15)
 				)
 			)
@@
 				(font
 					(size 0.001 0.001)
+					(thickness 0.15)
 				)
 			)
@@
 				(font
 					(size 0.001 0.001)
+					(thickness 0.15)
 				)
 			)
@@
 				(font
 					(size 0.001 0.001)
+					(thickness 0.15)
 				)
 			)
@@
 	(footprint "SparkFun-Resistor:R_0402_1005Metric"
 		(layer "F.Cu")
-		(at 139.776 104.456 -90)
+		(at 141.046 106.6785 -90)
 		(descr "Resistor SMD 0402 (1005 Metric), square (rectangular) end terminal, IPC_7351 nominal, (Body size source: IPC-SM-782 page 72, https://www.pcb-3d.com/wordpress/wp-content/uploads/ipc-sm-782a_amendment_1_and_2.pdf), generated with kicad-footprint-generator")
 		(tags "SparkFun resistor")
@@
 				(font
 					(size 0.001 0.001)
+					(thickness 0.15)
 				)
 				(justify mirror)
@@
 				(font
 					(size 0.001 0.001)
+					(thickness 0.15)
 				)
 				(justify mirror)
@@
 				(font
 					(size 0.001 0.001)
+					(thickness 0.15)
 				)
 				(justify mirror)
@@
 				(font
 					(size 0.001 0.001)
+					(thickness 0.15)
 				)
 				(justify mirror)
@@
 				(font
 					(size 0.001 0.001)
+					(thickness 0.15)
 				)
 				(justify mirror)
@@
 				(font
 					(size 0.001 0.001)
+					(thickness 0.15)
 				)
 				(justify mirror)
@@
 				(font
 					(size 0.001 0.001)
+					(thickness 0.15)
 				)
 				(justify mirror)
@@
 				(font
 					(size 0.001 0.001)
+					(thickness 0.15)
 				)
 				(justify mirror)
@@
 				(font
 					(size 0.001 0.001)
+					(thickness 0.15)
 				)
 				(justify mirror)
@@
 				(font
 					(size 0.001 0.001)
+					(thickness 0.15)
 				)
 				(justify mirror)
@@
 	)
 	(segment
-		(start 134.624018 104.7735)
-		(end 134.665763 104.731755)
+		(start 141.3635 108.5835)
+		(end 142.316 109.536)
 		(width 0.1524)
 		(layer "F.Cu")
@@
 	)
 	(segment
-		(start 134.766 104.7035)
-		(end 134.766 103.8535)
+		(start 134.624018 104.7735)
+		(end 134.665763 104.731755)
 		(width 0.1524)
 		(layer "F.Cu")
@@
 	)
 	(segment
-		(start 141.046 106.996)
-		(end 141.046 108.266)
+		(start 134.766 104.7035)
+		(end 134.766 103.8535)
 		(width 0.1524)
 		(layer "F.Cu")
@@
 	)
 	(segment
-		(start 141.046 108.266)
-		(end 142.316 109.536)
+		(start 141.046 108.5835)
+		(end 141.3635 108.5835)
 		(width 0.1524)
 		(layer "F.Cu")
@@
 	)
 	(via
-		(at 141.046 106.996)
+		(at 141.046 108.5835)
 		(size 0.56)
 		(drill 0.3)
@@
 	)
 	(segment
-		(start 134.6198 105.6498)
-		(end 134.6198 104.846653)
+		(start 141.046 108.5835)
+		(end 139.4585 106.996)
 		(width 0.1524)
 		(layer "B.Cu")
@@
 	)
 	(segment
-		(start 141.046 106.996)
+		(start 139.4585 106.996)
 		(end 135.966 106.996)
 		(width 0.1524)
@@
 	)
 	(segment
+		(start 134.6198 105.6498)
+		(end 134.6198 104.846653)
+		(width 0.1524)
+		(layer "B.Cu")
+		(net 14)
+	)
+	(segment
 		(start 134.546647 104.7735)
 		(end 134.624018 104.7735)
@@
 	)
 	(segment
-		(start 139.901 105.091)
-		(end 141.681 105.091)
+		(start 141.046 107.1885)
+		(end 141.556 106.6785)
 		(width 0.1524)
 		(layer "F.Cu")
@@
 	)
 	(segment
-		(start 141.681 105.091)
+		(start 141.556 106.6785)
 		(end 143.2685 106.6785)
 		(width 0.1524)
 		(layer "F.Cu")
-		(net 29)
-	)
-	(segment
-		(start 139.776 104.966)
-		(end 139.901 105.091)
-		(width 0.1524)
-		(layer "F.Cu")

Commit message: Updated part libraries
Parts:
- Y1: value 3.579MHz -> 3.579545MHz
Changed lines of the file:
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@@
 			)
 		)
-		(property "Value" "3.579MHz"
+		(property "Value" "3.579545MHz"
 			(at 0 2.05 0)
 			(layer "F.Fab")
@@
 			)
 		)
-		(property "Datasheet" "https://abracon.com/datasheets/ASEDV.pdf"
+		(property "Datasheet" "https://mm.digikey.com/Volume0/opasdata/d220001/medias/docus/8913/SG-210STF_X1G0041710031_en.pdf"
 			(at 0 0 0)
 			(unlocked yes)
@@
 			)
 		)
-		(property "PROD_ID" "XTAL-25500"
+		(property "PROD_ID" "XTAL-28569"
 			(at 0 0 0)
 			(unlocked yes)
@@
 			)
 		)
+		(property "PROD_ID" "IC-28571"
+			(at 0 0 180)
+			(unlocked yes)
+			(layer "F.Fab")
+			(hide yes)
+			(effects
+				(font
+					(size 1 1)
+					(thickness 0.15)
+				)
+			)
+		)
 		(sheetname "/")
 		(sheetfile "SparkFun_Qwiic_Current_Sensor_ADE7953.kicad_sch")
@@
 			)
 		)
-		(property "PROD_ID" "RES-09823"
+		(property "PROD_ID" "RES-28570"
 			(at 0 0 0)
 			(unlocked yes)
@@
 			)
 		)
-		(property "PROD_ID" "RES-09823"
+		(property "PROD_ID" "RES-28570"
 			(at 0 0 0)
 			(unlocked yes)
@@
 			(keep_text_aligned yes)
 		)
-		(gr_text "900 mils"
+		(gr_text "22.86 mm"
 			(at 115.4461 99.376 90)
 			(layer "Dwgs.User")
@@
 			(keep_text_aligned yes)
 		)
-		(gr_text "1000 mils"
+		(gr_text "25.4 mm"
 			(at 113.2236 98.106 90)
 			(layer "Dwgs.User")
@@
 			(keep_text_aligned yes)
 		)
-		(gr_text "1000 mils"
+		(gr_text "25.4 mm"
 			(at 135.966 119.1786 0)
 			(layer "Dwgs.User")
@@
 			(keep_text_aligned yes)
 		)
-		(gr_text "900 mils"
+		(gr_text "22.86 mm"
 			(at 134.696 116.6386 0)
 			(layer "Dwgs.User")
@@
 			(extension_offset 0.5)
 		)
-		(gr_text "100 mils"
+		(gr_text "2.54 mm"
 			(at 139.4585 114.13975 0)
 			(layer "Dwgs.User")
@@
 			(extension_offset 0.5)
 		)
-		(gr_text "500 mils"
+		(gr_text "12.7 mm"
 			(at 117.6686 104.456 90)
 			(layer "Dwgs.User")
@@
 			(keep_text_aligned yes)
 		)
-		(gr_text "100 mils"
+		(gr_text "2.54 mm"
 			(at 121.361 100.9635 90)
 			(layer "Dwgs.User")
@@
 			(keep_text_aligned yes)
 		)
-		(gr_text "250 mils"
+		(gr_text "6.35 mm"
 			(at 128.981 115.886 0)
 			(layer "Dwgs.User")
