File: Hardware/SparkFun_Qwiic_Current_Sensor_ADE7953.kicad_pcb (KiCad board)
At the start: 2 copper layers, 25.4 x 25.4 mm, 86 parts, among them J1 Qwiic_RA, J2 Qwiic_RA, J3 Conn_01x06, J4 Conn_01x02, J5 3.5mm TRRS, J6 Conn_01x02, U1 ADE7953ACPZ, Y1 3.579545MHz

Commit message: Updated PCB to v1.1
Parts:
- removed kibuzzard-689A6711: G***, kibuzzard-689A6711
- removed kibuzzard-689A6718: G***, kibuzzard-689A6718
- removed kibuzzard-69FCDE6F: G***, kibuzzard-69FCDE6F
- added kibuzzard-6A8F671A: G***, kibuzzard-6A8F671A, B.Cu at (145.8, 103.8)
- added kibuzzard-6A8F6918: G***, kibuzzard-6A8F6918, B.Cu at (134.7, 107.0)
- added kibuzzard-6A8F6922: G***, kibuzzard-6A8F6922, B.Cu at (137.2, 107.0)
Other:
- board text added: "v11"
- board text removed: "v10"
